File: hexagon/hexagon--.kicad_pcb (KiCad board)
At the start: 2 copper layers, 100 x 86.6 mm, 31 parts, among them J1 Conn_01x05_Pin, J2 Conn_01x05_Pin, J3 Conn_01x05_Pin, J4 Conn_01x05_Pin, J5 Conn_01x05_Pin, J6 Conn_01x05_Pin

Commit message: great success!
Parts:
- removed C2, C4, C8: C, Capacitor_SMD:C_0805_2012Metric_Pad1.18x1.45mm_HandSolder
Routing:
- net GND: track 523.1 -> 501.8 mm
- net +5V: track 427.5 -> 422.7 mm
Other:
- outline, holes or cut-outs redrawn
