File: square/square++.kicad_pcb (KiCad board)
At the start: 2 copper layers, 50 x 50 mm, 25 parts, among them J1 Conn_01x05_Pin, J2 Conn_01x05_Pin, J3 Conn_01x05_Pin, J4 Conn_01x05_Pin

Commit message: great success!
Parts:
- removed the JP1 at (189.5, 107.9)
- removed the JP1 at (157.9, 110.0)
- removed the JP1 at (160.0, 142.3)
- removed the JP1 at (192.2, 139.2)
Routing:
- net Net-(D8-DOUT): track 46.2 -> 43.0 mm
- net Net-(D1-DOUT): track 14.1 -> 11.5 mm
- net Net-(D6-DOUT): track 14.8 -> 12.2 mm
- net Net-(D4-DOUT): track 14.7 -> 12.2 mm
- net Net-(D5-DOUT): track 12.9 -> 10.5 mm
- net Net-(D3-DOUT): track 12.9 -> 10.5 mm
- net Net-(D2-DOUT): track 15.5 -> 13.2 mm
- net Net-(D7-DOUT): track 13.0 -> 11.0 mm
Other:
- outline, holes or cut-outs redrawn
