File: sq-half/sq-half--.kicad_pcb (KiCad board)
At the start: 2 copper layers, 50 x 50 mm, 11 parts, among them J1 Conn_01x05_Pin, J2 Conn_01x05_Pin, J3 Conn_01x05_Pin, J4 Conn_01x05_Pin

Commit message: updated all coolness
Parts:
- moved C1 8.80 mm to (21.6, 61.0)
- moved D1 0.60 mm to (17.8, 60.4)
- moved D4 0.60 mm to (60.0, 60.6)
- moved D2 0.60 mm to (18.0, 18.2)
- moved D3 0.60 mm to (60.2, 18.4)
Routing:
- net GND: track 197.4 -> 205.7 mm
- net +5V: track 195.1 -> 200.2 mm
- net Net-(D1-DIN): track 21.7 -> 20.9 mm
- net Net-(D4-DOUT): track 44.2 -> 43.6 mm
- net Net-(D3-DOUT): track 45.3 -> 44.7 mm
Other:
- outline, holes or cut-outs redrawn
