File: decagon/decagon--.kicad_pcb (KiCad board)
At the start: 2 copper layers, 161.7 x 153.8 mm, 39 parts, among them J1 Conn_01x05_Pin, J10 Conn_01x05_Pin, J2 Conn_01x05_Pin, J3 Conn_01x05_Pin, J4 Conn_01x05_Pin, J5 Conn_01x05_Pin, J6 Conn_01x05_Pin, J7 Conn_01x05_Pin, J8 Conn_01x05_Pin, J9 Conn_01x05_Pin

Commit message: very nice
Changed lines of the file:
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@@
 		(tags "Through hole pin header THT 1x05 2.54mm single row")
 		(property "Reference" "J6"
-			(at 0.000001 -2.379999 126)
+			(at 0 -2.379999 126)
 			(layer "F.SilkS")
 			(effects
@@
 		(tags "Through hole pin header THT 1x05 2.54mm single row")
 		(property "Reference" "J1"
-			(at 0.000001 -2.379999 126)
+			(at 0 -2.379999 126)
 			(layer "F.SilkS")
 			(effects
@@
 		)
 		(fp_line
-			(start -1.38 1.27)
+			(start -1.380001 1.27)
 			(end -1.380002 11.540002)
 			(stroke
@@
 		)
 		(fp_line
-			(start -1.38 1.27)
+			(start -1.380001 1.27)
 			(end 1.38 1.27)
 			(stroke
@@
 		(tags "LED RGB NeoPixel PLCC-4 5050")
 		(property "Reference" "D4"
-			(at 0 -3.5 72)
+			(at -0.000001 -3.5 72)
 			(layer "F.SilkS")
 			(effects
@@
 		)
 		(fp_line
-			(start -3.5 -2.3)
+			(start -3.5 -2.299999)
 			(end -3.5 2.75)
 			(stroke
@@
 		(fp_line
 			(start -3.050001 -2.750004)
-			(end -3.5 -2.3)
+			(end -3.5 -2.299999)
 			(stroke
 				(width 0.12)
@@
 		(tags "LED RGB NeoPixel PLCC-4 5050")
 		(property "Reference" "D14"
-			(at 0 -3.5 72)
+			(at -0.000001 -3.5 72)
 			(layer "F.SilkS")
 			(effects
@@
 		(fp_line
 			(start -3.050001 -2.750004)
-			(end -3.5 -2.3)
+			(end -3.5 -2.299999)
 			(stroke
 				(width 0.12)
@@
 		)
 		(fp_line
-			(start -3.5 -2.3)
+			(start -3.5 -2.299999)
 			(end -3.5 2.75)
 			(stroke
@@
 		)
 		(fp_line
-			(start -1.38 1.27)
+			(start -1.380001 1.27)
 			(end 1.38 1.27)
 			(stroke
@@
 		)
 		(fp_line
-			(start -1.38 1.27)
+			(start -1.380001 1.27)
 			(end -1.380002 11.540002)
 			(stroke
@@
 		(tags "LED RGB NeoPixel PLCC-4 5050")
 		(property "Reference" "D5"
-			(at 0 -3.5 162)
+			(at -0.000001 -3.5 162)
 			(layer "F.SilkS")
 			(effects
@@
 		(attr smd)
 		(fp_line
-			(start -3.5 -2.3)
+			(start -3.5 -2.299999)
 			(end -3.5 2.75)
 			(stroke
@@
 		(fp_line
 			(start -3.050001 -2.750004)
-			(end -3.5 -2.3)
+			(end -3.5 -2.299999)
 			(stroke
 				(width 0.12)
@@
 		(tags "LED RGB NeoPixel PLCC-4 5050")
 		(property "Reference" "D15"
-			(at 0 -3.5 162)
+			(at -0.000001 -3.5 162)
 			(layer "F.SilkS")
 			(effects
@@
 		(fp_line
 			(start -3.050001 -2.750004)
-			(end -3.5 -2.3)
+			(end -3.5 -2.299999)
 			(stroke
 				(width 0.12)
@@
 		)
 		(fp_line
-			(start -3.5 -2.3)
+			(start -3.5 -2.299999)
 			(end -3.5 2.75)
 			(stroke
